File: SampleCircuit.kicad_pcb (KiCad board)
At the start: 2 copper layers, 100 x 90 mm, 50 parts, among them J1 24V INPUT, J2 12V TEST, J3 5V TEST, J4 3.3V TEST, J5 SPEAKER, SW1 RESET, SW2 BOOT, U1 LMZM23601SILR, U15 TLV803S, U2 ESP32-S3-WROOM-1, U23 RV-3028-C7, U24 LMZM23601SILR, U25 LMZM23601SILR, U5 NS4168, U6 MicroSD

Commit message: Complete routing: GND stitching vias, manual route 3 remaining nets
Add 8 GND stitching vias for isolated F.Cu pads, manually route
+3.3V to U23, Net-(D8-K) to C34, and Net-(U23-VBACKUP) to U23.
All nets now fully connected (385 tracks, 44 vias, 0 unrouted).
Add spec section 13h for unrouted net cleanup process.

Co-Authored-By: Claude Opus 4.6 <noreply@anthropic.com>
Parts:
- moved C34 1.40 mm to (158.6, 96.0), turned to 180 degrees
Routing:
- net Net-(D8-K): track 28.1 -> 48.6 mm, vias 0 -> 2
- net +3.3V: track 177.3 -> 193.2 mm
- net Net-(U23-VBACKUP): track 33.8 -> 38.4 mm
- net GND: track 0.00 -> 4.40 mm, vias 0 -> 10
Changed lines of the file:
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@@
 	(footprint "JLCImport:GRM32ER7YA106KA12L"
 		(layer "F.Cu")
-		(at 160 96 90)
+		(at 158.6 96 180)
 		(descr "GRM32ER7YA106KA12L; C1210; muRata")
 		(tags "C1210 C97973 GRM32ER7YA106KA12L muRata")
 		(property "Reference" "C34"
-			(at 3.439802 0 0)
+			(at 3.439802 0 90)
 			(layer "F.SilkS")
 			(effects
@@
 		)
 		(property "Value" "10uF 35V"
-			(at 0 2.578613 90)
+			(at 0 2.578613 0)
 			(layer "F.Fab")
 			(hide yes)
@@
 		)
 		(property "Datasheet" ""
-			(at 0 0 90)
+			(at 0 0 0)
 			(layer "F.Fab")
 			(hide yes)
@@
 		)
 		(property "Description" ""
-			(at 0 0 90)
+			(at 0 0 0)
 			(layer "F.Fab")
 			(hide yes)
@@
 		(attr smd)
 		(fp_line
-			(start -2.411201 -1.578613)
-			(end -0.776199 -1.578613)
+			(start 2.563602 1.426213)
+			(end 2.563602 -1.426212)
 			(stroke
 				(width 0.1524)
@@
 		)
 		(fp_line
-			(start -2.563602 1.426212)
-			(end -2.563602 -1.426213)
+			(start 0.776199 1.578613)
+			(end 2.411201 1.578613)
 			(stroke
 				(width 0.1524)
@@
 		)
 		(fp_line
-			(start 2.563602 1.426213)
-			(end 2.563602 -1.426212)
+			(start -0.7762 1.578613)
+			(end -2.411201 1.578612)
 			(stroke
 				(width 0.1524)
@@
 		)
 		(fp_line
-			(start 0.776199 1.578613)
-			(end 2.411201 1.578613)
+			(start -2.411201 -1.578613)
+			(end -0.776199 -1.578613)
 			(stroke
 				(width 0.1524)
@@
 		)
 		(fp_line
-			(start -0.7762 1.578613)
-			(end -2.411201 1.578612)
+			(start -2.563602 1.426212)
+			(end -2.563602 -1.426213)
 			(stroke
 				(width 0.1524)
@@
 		)
 		(fp_arc
-			(start 2.411201 -1.578612)
-			(mid 2.518965 -1.533975)
-			(end 2.563602 -1.426212)
+			(start 2.563602 1.426213)
+			(mid 2.518965 1.533976)
+			(end 2.411201 1.578613)
 			(stroke
 				(width 0.1524)
@@
 		)
 		(fp_arc
-			(start -2.563602 -1.426213)
-			(mid -2.518965 -1.533976)
-			(end -2.411201 -1.578613)
+			(start 2.411201 -1.578612)
+			(mid 2.518965 -1.533975)
+			(end 2.563602 -1.426212)
 			(stroke
 				(width 0.1524)
@@
 		)
 		(fp_arc
-			(start 2.563602 1.426213)
-			(mid 2.518965 1.533976)
-			(end 2.411201 1.578613)
+			(start -2.411201 1.578612)
+			(mid -2.518965 1.533975)
+			(end -2.563602 1.426212)
 			(stroke
 				(width 0.1524)
@@
 		)
 		(fp_arc
-			(start -2.411201 1.578612)
-			(mid -2.518965 1.533975)
-			(end -2.563602 1.426212)
+			(start -2.563602 -1.426213)
+			(mid -2.518965 -1.533976)
+			(end -2.411201 -1.578613)
 			(stroke
 				(width 0.1524)
@@
 		)
 		(pad "1" smd rect
-			(at -1.517399 0 90)
+			(at -1.517399 0 180)
 			(size 1.635001 2.7)
 			(layers "F.Cu" "F.Mask" "F.Paste")
@@
 		)
 		(pad "2" smd rect
-			(at 1.517399 0 90)
+			(at 1.517399 0 180)
 			(size 1.635001 2.7)
 			(layers "F.Cu" "F.Mask" "F.Paste")
@@
 	)
 	(segment
+		(start 145 108)
+		(end 145 106.9)
+		(width 0.2)
+		(layer "F.Cu")
+		(net 2)
+	)
+	(via
+		(at 162.1 113.9)
+		(size 0.6)
+		(drill 0.3)
+		(layers "F.Cu" "B.Cu")
+		(tenting front back)
+		(net 2)
+	)
+	(via
+		(at 145 106.9)
+		(size 0.6)
+		(drill 0.3)
+		(layers "F.Cu" "B.Cu")
+		(net 2)
+	)
+	(via
+		(at 155.8 100)
+		(size 0.6)
+		(drill 0.3)
+		(layers "F.Cu" "B.Cu")
+		(tenting front back)
+		(net 2)
+	)
+	(via
+		(at 150.8 81)
+		(size 0.6)
+		(drill 0.3)
+		(layers "F.Cu" "B.Cu")
+		(tenting front back)
+		(net 2)
+	)
+	(via
+		(at 141 108.8)
+		(size 0.6)
+		(drill 0.3)
+		(layers "F.Cu" "B.Cu")
+		(tenting front back)
+		(net 2)
+	)
+	(via
+		(at 130.8 81)
+		(size 0.6)
+		(drill 0.3)
+		(layers "F.Cu" "B.Cu")
+		(tenting front back)
+		(net 2)
+	)
+	(via
+		(at 115.8 81)
+		(size 0.6)
+		(drill 0.3)
+		(layers "F.Cu" "B.Cu")
+		(tenting front back)
+		(net 2)
+	)
+	(via
+		(at 145 105.8)
+		(size 0.6)
+		(drill 0.3)
+		(layers "F.Cu" "B.Cu")
+		(tenting front back)
+		(net 2)
+	)
+	(via
+		(at 145 103.6)
+		(size 0.6)
+		(drill 0.3)
+		(layers "F.Cu" "B.Cu")
+		(net 2)
+	)
+	(via
+		(at 164.8 79)
+		(size 0.6)
+		(drill 0.3)
+		(layers "F.Cu" "B.Cu")
+		(tenting front back)
+		(net 2)
+	)
+	(segment
+		(start 145 106.9)
+		(end 145 103.6)
+		(width 0.2)
+		(layer "B.Cu")
+		(net 2)
+	)
+	(segment
 		(start 115 77.525)
 		(end 115 76.9116)
@@
 	)
 	(segment
+		(start 159.549911 99.342393)
+		(end 159.549911 98.742393)
+		(width 0.2)
+		(layer "F.Cu")
+		(net 4)
+	)
+	(segment
 		(start 141.4322 106.1267)
 		(end 143 106.1267)
@@
 	)
 	(segment
+		(start 151.1 98.3)
+		(end 151 98.4)
+		(width 0.2)
+		(layer "F.Cu")
+		(net 4)
+	)
+	(segment
 		(start 139 98)
 		(end 139 97.5991)
@@
 	)
 	(segment
+		(start 159.107518 98.3)
+		(end 151.1 98.3)
+		(width 0.2)
+		(layer "F.Cu")
+		(net 4)
+	)
+	(segment
 		(start 146.7423 84.018)
 		(end 147 84.018)
@@
 	)
 	(segment
+		(start 159.549911 98.742393)
+		(end 159.107518 98.3)
+		(width 0.2)
+		(layer "F.Cu")
+		(net 4)
+	)
+	(segment
 		(start 143 108)
 		(end 143 106.1267)
@@
 	)
 	(segment
+		(start 151 98.4)
+		(end 151 105)
+		(width 0.2)
+		(layer "F.Cu")
+		(net 4)
+	)
+	(segment
 		(start 172.0852 110.5001)
 		(end 172.9063 111.3212)
@@
 	)
 	(segment
+		(start 157.082601 96)
+		(end 153.9 96)
+		(width 0.2)
+		(layer "F.Cu")
+		(net 7)
+	)
+	(segment
 		(start 147.9128 77.3562)
 		(end 148.4707 76.7983)
@@
 	)
 	(segment
+		(start 160.794971 89.6)
+		(end 164.394971 86)
+		(width 0.2)
+		(layer "F.Cu")
+		(net 7)
+	)
+	(segment
+		(start 157.9 89.6)
+		(end 160.794971 89.6)
+		(width 0.2)
+		(layer "F.Cu")
+		(net 7)
+	)
+	(segment
 		(start 150 76.7998)
 		(end 150 76.7983)
@@
 	)
 	(segment
+		(start 153.9 96)
+		(end 152.6 94.7)
+		(width 0.2)
+		(layer "F.Cu")
+		(net 7)
+	)
+	(segment
 		(start 156.0043 76.7983)
 		(end 163.9793 84.7733)
@@
 		(net 7)
 	)
+	(via
+		(at 157.9 89.6)
+		(size 0.6)
+		(drill 0.3)
+		(layers "F.Cu" "B.Cu")
+		(net 7)
+	)
+	(via
+		(at 152.6 94.7)
+		(size 0.6)
+		(drill 0.3)
+		(layers "F.Cu" "B.Cu")
+		(net 7)
+	)
+	(segment
+		(start 157.7 89.6)
+		(end 157.9 89.6)
+		(width 0.2)
+		(layer "B.Cu")
+		(net 7)
+	)
+	(segment
+		(start 152.6 94.7)
+		(end 157.7 89.6)
+		(width 0.2)
+		(layer "B.Cu")
+		(net 7)
+	)
 	(segment
 		(start 138.3697 99.767)
@@
 	)
 	(segment
+		(start 160.6 98.3)
+		(end 162 98.3)
+		(width 0.2)
+		(layer "F.Cu")
+		(net 9)
+	)
+	(segment
+		(start 160.450089 98.449911)
+		(end 160.6 98.3)
+		(width 0.2)
+		(layer "F.Cu")
+		(net 9)
+	)
+	(segment
 		(start 138.3422 92.9409)
 		(end 138 93.2831)
@@
 	)
 	(segment
+		(start 163 99.3)
+		(end 163 100)
+		(width 0.2)
+		(layer "F.Cu")
+		(net 9)
+	)
+	(segment
 		(start 163 100)
 		(end 163 94.8164)
@@
 	)
 	(segment
+		(start 160.450089 99.342393)
+		(end 160.450089 98.449911)
+		(width 0.2)
+		(layer "F.Cu")
+		(net 9)
+	)
+	(segment
 		(start 138 93.2831)
 		(end 138 96)
@@
 		(layer "F.Cu")
 		(net 9)
+	)
+	(segment
+		(start 162 98.3)
+		(end 163 99.3)
+		(width 0.2)
+		(layer "F.Cu")
+		(net 9)
